File: pcb_utility_dc/pcb_utility_dc/pcb_utility_dc.kicad_pcb (KiCad board)
At the start: 2 copper layers, 5 parts, among them J1 Barrel_Jack_Switch, J2 Conn_01x02, Q1 MCH6341-TL-W

Commit message: us8 based switching files
Parts:
- J1: footprint Connectors_Jacks_DC:Jack_DC -> Connectors_Jacks_DC:Jack_DC_Mirrored
Changed lines of the file:
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@@
     (add_net "Net-(Q1-PadD)")
-  )
-  (module Connectors_Jacks_DC:Jack_DC (layer F.Cu)
-    (at 148.5 106.5)
-    (descr $KICAD_MYGITHUBDATASHEETS$\Connectors_Jacks_DC\A-2237.pdf)
-    (fp_text reference J1 (at 0 5) (layer F.SilkS) hide
-      (effects (font (size 0.8 0.8) (thickness 0.15)))
-    )
-    (fp_text value Barrel_Jack_Switch (at 0 6.5) (layer F.Fab)
-      (effects (font (size 0.8 0.8) (thickness 0.15)))
-    )
-    (fp_circle (center 0 0) (end 7 0) (layer F.CrtYd) (width 0.12))
-    (fp_circle (center 0 -2) (end 0 -5.15) (layer F.CrtYd) (width 0.12))
-    (fp_line (start 0 -2) (end 0.5 -2.5) (layer F.CrtYd) (width 0.12))
-    (fp_line (start 0.5 -2.5) (end 0 -2) (layer F.CrtYd) (width 0.12))
-    (fp_line (start 0 -2) (end 0.5 -1.5) (layer F.CrtYd) (width 0.12))
-    (fp_line (start 0.5 -1.5) (end 0 -2) (layer F.CrtYd) (width 0.12))
-    (fp_line (start 0 -2) (end -0.5 -1.5) (layer F.CrtYd) (width 0.12))
-    (fp_line (start -0.5 -1.5) (end 0 -2) (layer F.CrtYd) (width 0.12))
-    (fp_line (start 0 -2) (end -0.5 -2.5) (layer F.CrtYd) (width 0.12))
-    (fp_line (start 0 0) (end -0.5 -0.5) (layer F.CrtYd) (width 0.12))
-    (fp_line (start 0.5 -0.5) (end -0.5 0.5) (layer F.CrtYd) (width 0.12))
-    (fp_line (start 0 0) (end 0.5 0.5) (layer F.CrtYd) (width 0.12))
-    (pad 1 thru_hole oval (at -3.7 -2) (size 1.6 4.5) (drill oval 0.8 3) (layers *.Cu *.Mask)
-      (net 3 "Net-(J1-Pad1)"))
-    (pad 2 thru_hole oval (at -1.7 3.3) (size 4.5 1.6) (drill oval 3 0.8) (layers *.Cu *.Mask)
-      (net 2 "Net-(J1-Pad2)"))
-    (pad 3 thru_hole oval (at 1.7 1.4) (size 4.5 1.6) (drill oval 3 0.8) (layers *.Cu *.Mask)
-      (net 1 "Net-(J1-Pad3)"))
   )
   (module Connector_Wire:SolderWirePad_1x02_P3.81mm_Drill0.8mm (layer F.Cu)
@@
     )
   )
+  (module Connectors_Jacks_DC:Jack_DC_Mirrored (layer F.Cu)
+    (at 148.5 106.5)
+    (descr $KICAD_MYGITHUBDATASHEETS$\Connectors_Jacks_DC\A-2237.pdf)
+    (fp_text reference J1 (at 0 5) (layer F.SilkS) hide
+      (effects (font (size 1 1) (thickness 0.15)))
+    )
+    (fp_text value Barrel_Jack_Switch (at 0 6.5) (layer F.Fab)
+      (effects (font (size 1 1) (thickness 0.15)))
+    )
+    (fp_circle (center 0 0) (end -7 0) (layer F.CrtYd) (width 0.12))
+    (fp_circle (center 0 -2) (end 0 -5.15) (layer F.CrtYd) (width 0.12))
+    (fp_line (start 0 -2) (end -0.5 -2.5) (layer F.CrtYd) (width 0.12))
+    (fp_line (start -0.5 -2.5) (end 0 -2) (layer F.CrtYd) (width 0.12))
+    (fp_line (start 0 -2) (end -0.5 -1.5) (layer F.CrtYd) (width 0.12))
+    (fp_line (start -0.5 -1.5) (end 0 -2) (layer F.CrtYd) (width 0.12))
+    (fp_line (start 0 -2) (end 0.5 -1.5) (layer F.CrtYd) (width 0.12))
+    (fp_line (start 0.5 -1.5) (end 0 -2) (layer F.CrtYd) (width 0.12))
+    (fp_line (start 0 -2) (end 0.5 -2.5) (layer F.CrtYd) (width 0.12))
+    (fp_line (start 0 0) (end 0.5 -0.5) (layer F.CrtYd) (width 0.12))
+    (fp_line (start -0.5 -0.5) (end 0.5 0.5) (layer F.CrtYd) (width 0.12))
+    (fp_line (start 0 0) (end -0.5 0.5) (layer F.CrtYd) (width 0.12))
+    (pad 3 thru_hole oval (at 3.7 -2) (size 1.6 4.5) (drill oval 0.8 3) (layers *.Cu *.Mask)
+      (net 1 "Net-(J1-Pad3)"))
+    (pad 2 thru_hole oval (at 1.7 3.3) (size 4.5 1.6) (drill oval 3 0.8) (layers *.Cu *.Mask)
+      (net 2 "Net-(J1-Pad2)"))
+    (pad 1 thru_hole oval (at -1.7 1.4) (size 4.5 1.6) (drill oval 3 0.8) (layers *.Cu *.Mask)
+      (net 3 "Net-(J1-Pad1)"))
+  )
   (gr_text "Schematic:\n1 = GND\n2 = VCC\n3 = SW" (at 159 105.75) (layer Cmts.User)
