File: pcb_breakout_sm8_dct/pcb_breakout_sm8_dct.sch (KiCad schematic (older format))
At the start: 2 parts, among them J1 Conn_02x04_Counter_Clockwise, J2 Conn_02x04_Counter_Clockwise

Commit message: dct us8 breakout
Connections:
- net at J1.1 (Pin_1): now also J2.1 (Pin_1)
- net at J1.2 (Pin_2): now also J2.2 (Pin_2)
- net at J1.3 (Pin_3): now also J2.3 (Pin_3)
- net at J1.4 (Pin_4): now also J2.4 (Pin_4)
- net at J1.5 (Pin_5): now also J2.5 (Pin_5)
- net at J1.6 (Pin_6): now also J2.6 (Pin_6)
- net at J1.7 (Pin_7): now also J2.7 (Pin_7)
- net at J1.8 (Pin_8): now also J2.8 (Pin_8)
Changed lines of the file:
@@
 EESchema Schematic File Version 4
+LIBS:pcb_breakout_sm8_dct-cache
 EELAYER 29 0
 EELAYER END
@@
 	1    0    0    -1
 $EndComp
+Wire Wire Line
+	5450 4200 5350 4200
+Wire Wire Line
+	5350 4200 5350 4850
+Wire Wire Line
+	5350 4850 5450 4850
+Wire Wire Line
+	5450 4300 5250 4300
+Wire Wire Line
+	5250 4300 5250 4950
+Wire Wire Line
+	5250 4950 5450 4950
+Wire Wire Line
+	5450 4400 5150 4400
+Wire Wire Line
+	5150 4400 5150 5050
+Wire Wire Line
+	5150 5050 5450 5050
+Wire Wire Line
+	5450 4500 5050 4500
+Wire Wire Line
+	5050 4500 5050 5150
+Wire Wire Line
+	5050 5150 5450 5150
+Wire Wire Line
+	5950 4200 6050 4200
+Wire Wire Line
+	6050 4200 6050 4850
+Wire Wire Line
+	6050 4850 5950 4850
+Wire Wire Line
+	5950 4300 6150 4300
+Wire Wire Line
+	6150 4300 6150 4950
+Wire Wire Line
+	6150 4950 5950 4950
+Wire Wire Line
+	5950 4400 6250 4400
+Wire Wire Line
+	6250 5050 5950 5050
+Wire Wire Line
+	6250 4400 6250 5050
+Wire Wire Line
+	5950 4500 6350 4500
+Wire Wire Line
+	6350 4500 6350 5150
+Wire Wire Line
+	6350 5150 5950 5150
 $EndSCHEMATC

Commit message: cache changes
Parts:
- J1, J2: symbol Connector_Generic:Conn_02x04_Counter_Clockwise -> pcb_breakout_sm8_dct-rescue:Conn_02x04_Counter_Clockwise-Connector_Generic
Changed lines of the file:
@@
 EESchema Schematic File Version 4
 LIBS:pcb_breakout_sm8_dct-cache
-EELAYER 29 0
+EELAYER 26 0
 EELAYER END
 $Descr A4 11693 8268
@@
 $EndDescr
 $Comp
-L Connector_Generic:Conn_02x04_Counter_Clockwise J1
+L pcb_breakout_sm8_dct-rescue:Conn_02x04_Counter_Clockwise-Connector_Generic J1
 U 1 1 5C0DA4DE
 P 5650 4300
@@
 $EndComp
 $Comp
-L Connector_Generic:Conn_02x04_Counter_Clockwise J2
+L pcb_breakout_sm8_dct-rescue:Conn_02x04_Counter_Clockwise-Connector_Generic J2
 U 1 1 5C0DA678
 P 5650 4950
