File: Breadboard_Breakout_Boards/ON_Semi_MBT3946DW1T1G/ON_Semi_MBT3946DW1T1G.kicad_pcb (KiCad board)
At the start: 2 copper layers, 9.9 x 7.4 mm, 3 parts, among them J1 PinHeader_1x03_P2.54mm_Vertic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, J2 PinHeader_1x03_P2.54mm_Vertic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, Q1 ON_Semi_MCH6341-TL-W

Commit message: Breakout and utility boards
Parts:
- Q1: value ON_Semi_MCH6341-TL-W -> ON_Semi_MBT3946DW1T1G; footprint SA_Transistors_MOSFET_SMD:ON_Semi_MCH6341-TL-W_SOT-363_SC-70-6_SC-88 -> SA_Transistors_BJT_SMD:ON_Semi_MBT3946DW1T1G_SOT-363_SC-70-6_SC-80
Connections:
- J1 pad 1: /D -> /NE
- J1 pad 2: /D -> /NB
- J1 pad 3: /G -> /PC
- J2 pad 1: /D -> /NC
- J2 pad 2: /D -> /PB
- J2 pad 3: /S -> /PE
Routing:
- net /D: track 14.2 -> 0.00 mm
- net /S: track 4.36 -> 0.00 mm
- net /PE: track 0.00 -> 4.36 mm
- net /NC: track 0.00 -> 4.36 mm
- net /NE: track 0.00 -> 4.36 mm
- net /PC: track 0.00 -> 4.29 mm
- net /G: track 4.29 -> 0.00 mm
- net /PB: track 0.00 -> 2.76 mm
- net /NB: track 0.00 -> 2.76 mm
Other:
- board text added: "DW1T1G"
- board text added: "MBT3946"
- board text added: "NB"
- board text added: "NC"
- board text added: "NE"
- board text added: "PB"
- board text added: "PC"
- board text added: "PE"
- board text removed: "6341"
- board text removed: "MCH"
