File: Breadboard_Breakout_Boards/ON_Semi_NCP1117LPST50T3G/ON_Semi_NCP1117LPST50T3G.kicad_pcb (KiCad board)
At the start: 2 copper layers, 11.2 x 7.4 mm, 2 parts, among them J1 PinHeader_1x03_P2.54mm_Vertic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, U1 ON_Semi_NCP1117LPST50T3G

Commit message: Breakout and utility boards
Other:
- rule pad_to_mask_clearance: 0.051 -> 0.0508
- rule solder_mask_min_width: 0.25 -> 0.0508
Changed lines of the file:
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@@
     (pad_size 1.524 1.524)
     (pad_drill 0.762)
-    (pad_to_mask_clearance 0.051)
-    (solder_mask_min_width 0.25)
+    (pad_to_mask_clearance 0.0508)
+    (solder_mask_min_width 0.0508)
     (aux_axis_origin 0 0)
     (visible_elements 7FFFFFFF)
