File: Breadboard_Breakout_Boards/ON_Semi_NL37WZ14USG/ON_Semi_NL37WZ14USG.kicad_pcb (KiCad board)
At the start: 2 copper layers, 9.9 x 9.9 mm, 3 parts, among them J1 PinHeader_1x04_P2.54mm_Vertic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, J2 PinHeader_1x04_P2.54mm_Vertic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, U1 ON_Semi_NL37WZ14USG

Commit message: Breakout and utility boards
Other:
- rule pad_to_mask_clearance: 0.051 -> 0.0508
- rule solder_mask_min_width: 0.25 -> 0.0508
Changed lines of the file:
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@@
     (pad_size 1.7 1.7)
     (pad_drill 1)
-    (pad_to_mask_clearance 0.051)
-    (solder_mask_min_width 0.25)
+    (pad_to_mask_clearance 0.0508)
+    (solder_mask_min_width 0.0508)
     (aux_axis_origin 0 0)
     (visible_elements 7FFFFFFF)
