File: Breadboard_Breakout_Boards/Passives-1206-0805-0603/Passives-1206-0805-0603_0402_SOD-323_SMA.kicad_pcb (KiCad board)
At the start: 2 copper layers, 9.9 x 20.1 mm, 50 parts, among them J1 Conn_01x08, J2 Conn_01x08

Commit message: Breakout and utility boards
Changed lines of the file:
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@@
   (page A4)
   (layers
-    (0 F.Cu signal hide)
+    (0 F.Cu signal)
     (31 B.Cu signal)
     (32 B.Adhes user)
-    (33 F.Adhes user hide)
+    (33 F.Adhes user)
     (34 B.Paste user)
     (35 F.Paste user)
     (36 B.SilkS user)
-    (37 F.SilkS user hide)
+    (37 F.SilkS user)
     (38 B.Mask user)
-    (39 F.Mask user hide)
+    (39 F.Mask user)
     (40 Dwgs.User user)
     (41 Cmts.User user)
@@
     (solder_mask_min_width 0.0508)
     (aux_axis_origin 0 0)
-    (visible_elements 7FFF7DDF)
+    (visible_elements 7FFFFFFF)
     (pcbplotparams
       (layerselection 0x010ec_ffffffff)
@@
     (descr "Through hole straight pin header, 1x08, 2.54mm pitch, single row")
     (tags "Through hole pin header THT 1x08 2.54mm single row")
-    (fp_text reference J2 (at 0 -2.23) (layer F.SilkS)
+    (fp_text reference J2 (at 0 -2.23) (layer F.SilkS) hide
       (effects (font (size 0.6 0.6) (thickness 0.127)))
     )
@@
     (descr "Through hole straight pin header, 1x08, 2.54mm pitch, single row")
     (tags "Through hole pin header THT 1x08 2.54mm single row")
-    (fp_text reference J1 (at 0 -2.23) (layer F.SilkS)
+    (fp_text reference J1 (at 0 -2.23) (layer F.SilkS) hide
       (effects (font (size 0.6 0.6) (thickness 0.127)))
     )
