File: Breadboard_Breakout_Boards/Texas_Instruments_SN74LVC3G14DCTR/Texas_Instruments_SN74LVC3G14DCTR.kicad_pcb (KiCad board)
At the start: 2 copper layers, 9.9 x 9.9 mm, 3 parts, among them J1 PinHeader_1x04_P2.54mm_Vertic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, J2 PinHeader_1x04_P2.54mm_Vertic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, U1 Texas_Instruments_SN74LVC3G14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

Commit message: Breakout and utility boards
Other:
- rule pad_to_mask_clearance: 0.051 -> 0.0508
- rule solder_mask_min_width: 0.25 -> 0.0508
- board text added: "3G14DCTR"
- board text removed: "3G14"
Changed lines of the file:
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@@
     (pad_size 1.7 1.7)
     (pad_drill 1)
-    (pad_to_mask_clearance 0.051)
-    (solder_mask_min_width 0.25)
+    (pad_to_mask_clearance 0.0508)
+    (solder_mask_min_width 0.0508)
     (aux_axis_origin 0 0)
     (visible_elements 7FFFFFFF)
@@
     (at 128.27 95.25)
     (attr smd)
-    (fp_text reference U1 (at 0 -2.1) (layer F.SilkS)
+    (fp_text reference U1 (at 0 -2.1) (layer F.SilkS) hide
       (effects (font (size 0.6 0.6) (thickness 0.127)))
     )
@@
     (effects (font (size 0.6 0.6) (thickness 0.127)))
   )
-  (gr_text 3G14 (at 128.27 99.568) (layer F.Mask)
+  (gr_text 3G14DCTR (at 128.27 99.568) (layer F.Mask)
     (effects (font (size 0.6 0.6) (thickness 0.127)))
   )
-  (gr_text 3G14 (at 128.27 99.568) (layer F.Cu)
+  (gr_text 3G14DCTR (at 128.27 99.568) (layer F.Cu)
     (effects (font (size 0.6 0.6) (thickness 0.127)))
   )
