File: Utility_Boards/DC_Jack_Lumberg_Combined/Rev_A/DC_Jack_Lumberg_Combined.kicad_pcb (KiCad board)
At the start: 2 copper layers, 16.8 x 11.4 mm, 9 parts, among them J1 Lumberg_NEB_J_21_C, J2 Wire_Pad_2x, J3 Wire_Pad_2x

Commit message: Revision A boards checked before sending off to fab
Other:
- rule solder_mask_min_width: 0.0508 -> 0.25
Changed lines of the file:
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@@
   (general
     (thickness 1.6)
-    (drawings 17)
+    (drawings 20)
     (tracks 5)
     (zones 0)
@@
     (last_trace_width 0.25)
     (trace_clearance 0.1524)
-    (zone_clearance 0.254)
+    (zone_clearance 0.1524)
     (zone_45_only no)
     (trace_min 0.2)
@@
     (mod_text_size 1 1)
     (mod_text_width 0.15)
-    (pad_size 0.59 0.64)
-    (pad_drill 0)
+    (pad_size 3 3)
+    (pad_drill 3)
     (pad_to_mask_clearance 0.0508)
-    (solder_mask_min_width 0.0508)
+    (solder_mask_min_width 0.25)
     (aux_axis_origin 0 0)
     (visible_elements 7FFFFFFF)
@@
     (pad "" np_thru_hole circle (at 0 0) (size 1.75 1.75) (drill 1.75) (layers *.Cu *.Mask))
   )
+  (dimension 5.334 (width 0.3) (layer F.Fab)
+    (gr_text "5.334 mm" (at 177.106 98.425 90) (layer F.Fab)
+      (effects (font (size 1.5 1.5) (thickness 0.3)))
+    )
+    (feature1 (pts (xy 152.146 95.758) (xy 175.592421 95.758)))
+    (feature2 (pts (xy 152.146 101.092) (xy 175.592421 101.092)))
+    (crossbar (pts (xy 175.006 101.092) (xy 175.006 95.758)))
+    (arrow1a (pts (xy 175.006 95.758) (xy 175.592421 96.884504)))
+    (arrow1b (pts (xy 175.006 95.758) (xy 174.419579 96.884504)))
+    (arrow2a (pts (xy 175.006 101.092) (xy 175.592421 99.965496)))
+    (arrow2b (pts (xy 175.006 101.092) (xy 174.419579 99.965496)))
+  )
+  (dimension 2.667 (width 0.3) (layer F.Fab)
+    (gr_text "2.667 mm" (at 173.296 99.7585 90) (layer F.Fab)
+      (effects (font (size 1.5 1.5) (thickness 0.3)))
+    )
+    (feature1 (pts (xy 152.146 98.425) (xy 171.782421 98.425)))
+    (feature2 (pts (xy 152.146 101.092) (xy 171.782421 101.092)))
+    (crossbar (pts (xy 171.196 101.092) (xy 171.196 98.425)))
+    (arrow1a (pts (xy 171.196 98.425) (xy 171.782421 99.551504)))
+    (arrow1b (pts (xy 171.196 98.425) (xy 170.609579 99.551504)))
+    (arrow2a (pts (xy 171.196 101.092) (xy 171.782421 99.965496)))
+    (arrow2b (pts (xy 171.196 101.092) (xy 170.609579 99.965496)))
+  )
+  (dimension 2.54 (width 0.3) (layer F.Fab)
+    (gr_text "2.540 mm" (at 134.806 100.076 90) (layer F.Fab)
+      (effects (font (size 1.5 1.5) (thickness 0.3)))
+    )
+    (feature1 (pts (xy 142.367 98.806) (xy 136.319579 98.806)))
+    (feature2 (pts (xy 142.367 101.346) (xy 136.319579 101.346)))
+    (crossbar (pts (xy 136.906 101.346) (xy 136.906 98.806)))
+    (arrow1a (pts (xy 136.906 98.806) (xy 137.492421 99.932504)))
+    (arrow1b (pts (xy 136.906 98.806) (xy 136.319579 99.932504)))
+    (arrow2a (pts (xy 136.906 101.346) (xy 137.492421 100.219496)))
+    (arrow2b (pts (xy 136.906 101.346) (xy 136.319579 100.219496)))
+  )
   (dimension 11.430706 (width 0.3) (layer F.Fab)
     (gr_text "11.431 mm" (at 161.672093 97.471782 270.6365936) (layer F.Fab)
@@
   (segment (start 150.876 95.732) (end 148.082 95.732) (width 0.25) (layer B.Cu) (net 3))
   (zone (net 2) (net_name /DC+) (layer F.Cu) (hatch edge 0.508)
-    (connect_pads (clearance 0.254))
-    (min_thickness 0.254)
-    (fill yes (arc_segments 32) (thermal_gap 0.254) (thermal_bridge_width 0.255))
+    (connect_pads (clearance 0.1524))
+    (min_thickness 0.1524)
+    (fill yes (arc_segments 32) (thermal_gap 0.1524) (thermal_bridge_width 0.508))
     (polygon
       (pts
@@
   )
   (zone (net 3) (net_name /DC-) (layer B.Cu) (hatch edge 0.508)
-    (connect_pads (clearance 0.254))
-    (min_thickness 0.254)
-    (fill yes (arc_segments 32) (thermal_gap 0.254) (thermal_bridge_width 0.255))
+    (connect_pads (clearance 0.1524))
+    (min_thickness 0.1524)
+    (fill yes (arc_segments 32) (thermal_gap 0.1524) (thermal_bridge_width 0.254))
     (polygon
       (pts
