File: Utility_Boards/Neutrik_NRJ6HM-1/Rev_A/Neutrik_NRJ6HM-1.kicad_pcb (KiCad board)
At the start: 2 copper layers, 17.8 x 21.1 mm, 6 parts, among them J1 Neutrik_NRJ6HM-1_NoChassis, J2 Wire_Pad_3x

Commit message: Revision A boards checked before sending off to fab
Other:
- board text added: "3.0 mm NPTH for cable ties 1.2 mm PTH for wires"
Changed lines of the file:
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@@
   (general
     (thickness 1.6)
-    (drawings 15)
+    (drawings 16)
     (tracks 6)
     (zones 0)
@@
     (pad_drill 1.2)
     (pad_to_mask_clearance 0.051)
-    (solder_mask_min_width 0.25)
     (aux_axis_origin 0 0)
     (visible_elements 7FFFFFFF)
@@
     )
   )
+  (gr_text "3.0 mm NPTH for cable ties\n1.2 mm PTH for wires" (at 154.432 106.299) (layer F.Fab)
+    (effects (font (size 1.5 1.5) (thickness 0.3)) (justify left))
+  )
   (gr_line (start 171.577 89.408) (end 171.323 89.408) (layer B.Mask) (width 0.2))
