File: Utility_Boards/PCBA_RELAY/PCBA_RELAY.kicad_pcb (KiCad board)
At the start: 2 copper layers, 16.5 x 14 mm, 3 parts, among them J1 PinHeader_1x05_P2.54mm_Vertic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, J3 PinHeader_1x05_P2.54mm_Vertic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, K1 Kemet_EA2-5SNJ

Commit message: Cleanup
Other:
- board text added: "GND"
- board text added: "IN"
- board text added: "OUT"
- board text added: "RTN"
- board text added: "SND"
Changed lines of the file:
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@@
   (general
     (thickness 1.6)
-    (drawings 8)
+    (drawings 14)
     (tracks 24)
     (zones 0)
@@
     (fp_line (start -4.582289 7.102797) (end 4.617711 7.102797) (layer F.Fab) (width 0.15))
     (fp_line (start 4.617711 7.102797) (end 4.617711 -7.097203) (layer F.Fab) (width 0.15))
-    (fp_line (start 1.922711 -5.077203) (end -1.887289 -5.077203) (layer F.SilkS) (width 0.75))
+    (fp_line (start 1.922711 -5.077203) (end -1.887289 -5.077203) (layer F.Mask) (width 0.75))
     (pad 1 thru_hole roundrect (at -3.792289 -5.077203) (size 2 2) (drill 1.2) (layers *.Cu *.Mask) (roundrect_rratio 0.1)
       (net 6 /CAP_-))
@@
       (net 7 /SW_1))
   )
+  (gr_text RTN (at 128.27 102.87) (layer B.Mask)
+    (effects (font (size 0.6 0.6) (thickness 0.128)) (justify left mirror))
+  )
+  (gr_text IN (at 123.19 102.87) (layer B.Mask)
+    (effects (font (size 0.6 0.6) (thickness 0.128)) (justify right mirror))
+  )
+  (gr_text IN (at 128.27 97.79) (layer B.Mask)
+    (effects (font (size 0.6 0.6) (thickness 0.128)) (justify left mirror))
+  )
+  (gr_text OUT (at 128.27 100.33) (layer B.Mask)
+    (effects (font (size 0.6 0.6) (thickness 0.128)) (justify left mirror))
+  )
+  (gr_text SND (at 123.19 100.33) (layer B.Mask)
+    (effects (font (size 0.6 0.6) (thickness 0.128)) (justify right mirror))
+  )
+  (gr_text GND (at 123.19 97.79) (layer B.Mask)
+    (effects (font (size 0.6 0.6) (thickness 0.128)) (justify right mirror))
+  )
   (gr_arc (start 118.745 106.045) (end 117.475 106.045) (angle -90) (layer Edge.Cuts) (width 0.2))
