File: Utility_Boards/PCBA_SW/PCBA_SW.kicad_pcb (KiCad board)
At the start: 2 copper layers, 3 parts

Commit message: Cleanup
Parts:
- removed the REF** at (156.1, 71.8)
- removed the REF** at (167.9, 76.2)
- added REF**: PinHeader_1x02_P2.54mm_Vertical, Connector_PinHeader_2.54mm:PinHeader_1x02_P2.54mm_Vertical, F.Cu at (139.7, 76.2)
Routing:
- net (no net): track 0.00 -> 20.4 mm
Other:
- board outline added: 15.9 x 8.9 mm
- net class Default: clearance 0.2 -> 0.1524; trace_width 0.25 -> 0.508
- rule trace_clearance: 0.2 -> 0.1524
