File: Musitronics Mu-Tron II Phaser/LDR_Section.sch (KiCad schematic (older format))
At the start: 33 parts, among them U201 TL072, U202 TL072, U203 TL072

Commit message: mu-tron ii major work
Other:
- note added: "Connections:\n\n- VDD\n- VEE\n- GND\n\n- LDR IN/OUT"
