File: Musitronics Mu-Tron II Phaser/LFO_Section.sch (KiCad schematic (older format))
At the start: 27 parts, among them Q301 2N4401, U301 TL062, U302 TL072

Commit message: mu-tron ii major work
Parts:
- R311: value 3k9 -> 3k6
Other:
- note added: "Connections:\n-VDD\n-VEE\n-GND\n\n- Rate pot\n- Depth pot\n- LED"
- note added: "Tagboard layout has\n3 LED's in series"
- note added: "was 4k6"
- note added: "was 58k"
- moved on the sheet: R315, TR302
Changed lines of the file:
@@
 P 7050 4150
 F 0 "R311" V 7130 4150 50  0000 C CNN
-F 1 "3k9" V 7050 4150 50  0000 C CNN
+F 1 "3k6" V 7050 4150 50  0000 C CNN
 F 2 "" V 6980 4150 50  0001 C CNN
 F 3 "" H 7050 4150 50  0001 C CNN
@@
 L Mu-Tron-II-rescue:POT TR302
 U 1 1 5A7936DF
-P 8650 4450
-F 0 "TR302" V 8550 4450 50  0000 C CNN
-F 1 "1k" V 8650 4450 50  0000 C CNN
-F 2 "" H 8650 4450 50  0001 C CNN
-F 3 "" H 8650 4450 50  0001 C CNN
-	1    8650 4450
-	0    -1   -1   0
+P 8400 4700
+F 0 "TR302" V 8300 4700 50  0000 C CNN
+F 1 "1k" V 8400 4700 50  0000 C CNN
+F 2 "" H 8400 4700 50  0001 C CNN
+F 3 "" H 8400 4700 50  0001 C CNN
+	1    8400 4700
+	1    0    0    -1
 $EndComp
 $Comp
 L Device:R R315
 U 1 1 5A793805
-P 8900 4700
-F 0 "R315" V 8980 4700 50  0000 C CNN
-F 1 "390R" V 8900 4700 50  0000 C CNN
-F 2 "" V 8830 4700 50  0001 C CNN
-F 3 "" H 8900 4700 50  0001 C CNN
-	1    8900 4700
+P 8400 5100
+F 0 "R315" V 8480 5100 50  0000 C CNN
+F 1 "390R" V 8400 5100 50  0000 C CNN
+F 2 "" V 8330 5100 50  0001 C CNN
+F 3 "" H 8400 5100 50  0001 C CNN
+	1    8400 5100
 	1    0    0    -1
 $EndComp
@@
 	3650 3500 3750 3500
 Wire Wire Line
-	3750 2950 3750 3600
+	3750 2950 3750 3500
 Wire Wire Line
 	3750 2950 3500 2950
@@
 	3200 2950 2950 2950
 Wire Wire Line
-	2950 2750 2950 3400
+	2950 2750 2950 2950
 Wire Wire Line
 	2950 3400 3050 3400
@@
 	4500 3600 4400 3600
 Wire Wire Line
-	4400 3600 4400 4150
+	4400 3600 4400 3750
 Wire Wire Line
 	4400 3750 4300 3750
@@
 	5200 4150 4950 4150
 Wire Wire Line
-	5200 2750 5200 4550
-Wire Wire Line
-	5100 3500 5450 3500
+	5200 2750 5200 3500
+Wire Wire Line
+	5100 3500 5200 3500
 Wire Wire Line
 	4000 2750 2950 2750
@@
 	5450 4000 5450 3900
 Wire Wire Line
-	8400 4150 8400 4450
-Wire Wire Line
 	8100 3500 8000 3500
 Wire Wire Line
-	7300 3600 7300 4550
+	7300 3600 7300 4450
 Wire Wire Line
 	7300 3600 7400 3600
 Wire Wire Line
-	7300 4450 7800 4450
+	7300 4450 7550 4450
 Connection ~ 7300 4450
 Wire Wire Line
@@
 Connection ~ 7050 3400
 Wire Wire Line
-	8650 4300 8400 4300
-Connection ~ 8400 4300
-Connection ~ 8400 4450
-Wire Wire Line
-	8900 4550 8900 4450
-Wire Wire Line
-	8900 4450 8800 4450
-Wire Wire Line
-	6000 3750 5900 3750
+	6000 3750 5950 3750
 Wire Wire Line
 	5950 3750 5950 3400
@@
 	6750 3500 6750 4000
 Wire Wire Line
-	5950 3400 7400 3400
-Wire Wire Line
-	2950 5350 8900 5350
-Wire Wire Line
-	8900 5350 8900 4850
+	5950 3400 7050 3400
+Wire Wire Line
+	2950 5350 3750 5350
 Connection ~ 7550 5350
 Connection ~ 7050 5350
 Wire Wire Line
-	6450 4300 6450 5450
+	6450 4300 6450 5350
 Connection ~ 6450 5350
 Wire Wire Line
@@
 $EndComp
 Wire Wire Line
-	8100 4450 8500 4450
+	8100 4450 8400 4450
 $Comp
 L power:GND #PWR0306
@@
 Text Notes 8500 3900 0    60   ~ 12
 LED
+Wire Wire Line
+	3750 3500 3750 3600
+Wire Wire Line
+	4400 3750 4400 4150
+Wire Wire Line
+	2950 2950 2950 3400
+Wire Wire Line
+	5200 3500 5200 4150
+Wire Wire Line
+	5200 3500 5450 3500
+Wire Wire Line
+	5200 4150 5200 4550
+Wire Wire Line
+	7300 4450 7300 4550
+Wire Wire Line
+	7550 4450 7800 4450
+Wire Wire Line
+	7050 3400 7400 3400
+Wire Wire Line
+	5950 3750 5900 3750
+Wire Wire Line
+	7550 5350 8400 5350
+Wire Wire Line
+	7050 5350 7300 5350
+Wire Wire Line
+	6450 5350 7050 5350
+Wire Wire Line
+	6450 5350 6450 5450
+Wire Wire Line
+	5450 5350 6450 5350
+Wire Wire Line
+	5200 5350 5450 5350
+Wire Wire Line
+	3750 5350 5200 5350
+Wire Wire Line
+	7300 5350 7550 5350
+Text Notes 7000 4350 1    60   Italic 12
+was 4k6
+Text Notes 5550 3950 0    60   Italic 12
+was 58k
+Wire Wire Line
+	8400 4150 8400 4450
+Wire Wire Line
+	8400 4450 8400 4550
+Connection ~ 8400 4450
+Wire Wire Line
+	8400 4450 8550 4450
+Wire Wire Line
+	8550 4450 8550 4700
+Wire Wire Line
+	8400 4950 8400 4850
+Wire Wire Line
+	8400 5350 8400 5250
+Text Notes 8650 4250 0    60   Italic 12
+Tagboard layout has\n3 LED's in series
+Text Notes 5750 2550 0    60   Italic 12
+Connections:\n-VDD\n-VEE\n-GND\n\n- Rate pot\n- Depth pot\n- LED
 $EndSCHEMATC
