File: Musitronics Mu-Tron II Phaser/Power_Section.sch (KiCad schematic (older format))
At the start: 5 parts, among them J501 1044

Commit message: mu-tron ii major work
Changed lines of the file:
@@
 	6250 3750 6250 3950
 Wire Wire Line
-	6150 3950 6400 3950
+	6150 3950 6250 3950
 Wire Wire Line
 	6300 4350 6300 4250
 Wire Wire Line
-	6150 4250 6400 4250
+	6150 4250 6300 4250
 Connection ~ 6300 4250
 Connection ~ 6250 3950
@@
 	5650 4700 5650 4250
 Wire Wire Line
-	4950 4150 5650 4150
+	4950 4150 5250 4150
 Connection ~ 5250 4150
 $Comp
@@
 	5250 3650 4950 3650
 Wire Wire Line
-	4950 3550 4950 3750
+	4950 3550 4950 3650
 Connection ~ 4950 3650
+Wire Wire Line
+	6300 4250 6400 4250
+Wire Wire Line
+	6250 3950 6400 3950
+Wire Wire Line
+	5250 4150 5650 4150
+Wire Wire Line
+	4950 3650 4950 3750
 $EndSCHEMATC
