File: Musitronics Mu-Tron II Phaser/Layout Test/LDR Section/Mu-Tron II.kicad_pcb (KiCad board)
At the start: 2 copper layers, 31.8 x 30.5 mm, 36 parts, among them J201 Conn_01x08, J202 Conn_01x08, J205 Conn_01x03, U201 TL072, U202 TL072, U203 TL072

Commit message: mu-tron update, bom
Parts:
- added J205: Conn_01x03, Connector_PinHeader_1.27mm:PinHeader_1x03_P1.27mm_Vertical, F.Cu at (121.9, 81.3)
Connections:
- J201 pad 8: Net-(J201-Pad8) -> /LDR_Section/LDR_IN
- J202 pad 8: Net-(J202-Pad8) -> /LDR_Section/LDR_OUT
Routing:
- net /LDR_Section/LDR_IN: track 4.84 -> 35.8 mm
- net /LDR_Section/LDR_OUT: track 1.81 -> 29.7 mm, vias 0 -> 1
