File: Musitronics Mu-Tron II Phaser/Layout Test/Main Section/Main_Section.sch (KiCad schematic (older format))
At the start: 36 parts, among them J201 Conn_01x08, J202 Conn_01x08, J203 Conn_01x03, J204 Conn_01x03, J205 Conn_01x03, J206 Conn_01x03, J207 Conn_01x02, J208 Conn_01x03, U201 TL071, U202 TL072

Commit message: mu-tron update, bom
Parts:
- removed J207: Conn_01x02, Connector_PinHeader_1.27mm:PinHeader_1x02_P1.27mm_Vertical, symbol Connector_Generic:Conn_01x02
Connections:
- net LDR_IN: now also J201.8 (Pin_8)
- net LDR_OUT: now also J202.8 (Pin_8)
Changed lines of the file:
@@
 FX_OUT
-$Comp
-L Connector_Generic:Conn_01x02 J207
-U 1 1 5C93735D
-P 5950 5250
-F 0 "J207" H 5950 5350 50  0000 C CNN
-F 1 "Conn_01x02" H 5950 5050 50  0000 C CNN
-F 2 "Connector_PinHeader_1.27mm:PinHeader_1x02_P1.27mm_Vertical" H 5950 5250 50  0001 C CNN
-F 3 "~" H 5950 5250 50  0001 C CNN
-	1    5950 5250
-	-1   0    0    -1
-$EndComp
-Text HLabel 6150 5250 2    60   Input ~ 0
-LDR_IN
-Text HLabel 6150 5350 2    60   Input ~ 0
-LDR_OUT
 $Comp
 L Connector_Generic:Conn_01x03 J208
@@
 Wire Wire Line
 	2850 5800 2400 5800
+Text HLabel 7200 1800 2    60   Input ~ 0
+LDR_IN
+Text HLabel 7850 1800 2    60   Input ~ 0
+LDR_OUT
 $EndSCHEMATC
