File: Musitronics Mu-Tron II Phaser/Layout Test/Main Section/Mu-Tron II.kicad_pcb (KiCad board)
At the start: 2 copper layers, 31.8 x 47 mm, 38 parts, among them J201 Conn_01x08, J202 Conn_01x08, J203 Conn_01x03, J204 Conn_01x03, J208 Conn_01x03, J301 1044, U201 TL071, U202 TL072

Commit message: mu-tron update, bom
Parts:
- moved C206 1.80 mm to (127.0, 98.4)
Connections:
- J201 pad 8: Net-(J201-Pad8) -> /Main Section/LDR_IN
- J202 pad 8: Net-(J202-Pad8) -> /Main Section/LDR_OUT
Routing:
- net /Main Section/LDR_IN: track 3.71 -> 20.0 mm, vias 0 -> 1
- net /Main Section/LDR_OUT: track 0.00 -> 11.6 mm, vias 0 -> 2
- net VDD: track 69.5 -> 72.6 mm
- net Net-(C208-Pad1): track 33.1 -> 34.9 mm
- net Net-(C206-Pad1): track 6.18 -> 4.38 mm
- net Net-(R210-Pad2): track 8.01 -> 9.81 mm
- net Net-(R208-Pad2): track 8.29 -> 9.19 mm
- net Net-(C203-Pad1): track 21.5 -> 22.3 mm
- net Net-(J204-Pad2): track 36.7 -> 37.3 mm
- net Net-(J204-Pad3): track 37.2 -> 37.8 mm
- net Net-(J204-Pad1): track 36.2 -> 36.7 mm
