File: ValveWizard The Engineers Thumb [5 knob]/ValveWizard The Engineers Thumb [5 knob].kicad_pcb (KiCad board)
At the start: 2 copper layers, 109.7 x 84.1 mm, 46 parts, among them Q1 ON_Semi_2N3906TAR, SW1 SW_BRIGHT, U1 TL072, U2 TL072, U3 LM13700

Commit message: Projects upd
Parts:
- removed the REF** at (284.5, 58.4)
- removed the REF** at (210.8, 58.4)
- removed Taiwan_Alpha_RV16AF-10 (x5): VAL**, SA_Potentiometers_THT:Taiwan_Alpha_RV16AF-10
- RV1, RV2, RV3, RV4, RV5: footprint SA_Potentiometers_THT:Alpha_Taiwan_9mm_Vertical -> SA_Potentiometers_THT:Alpha_Taiwan_RV16AF-10_THT
- moved REF** 157.5 mm to (91.4, 83.8)
- moved R6 94.0 mm to (81.3, 68.6)
- moved RV5 91.5 mm to (50.8, 49.5)
- moved D4 89.6 mm to (76.2, 55.9)
- moved C5 89.6 mm to (86.4, 68.6), turned to 270 degrees
- moved C8 85.0 mm to (229.8, 58.8)
- moved RV3 84.3 mm to (71.1, 49.5)
- moved R4 82.5 mm to (111.8, 43.2)
- moved D3 82.3 mm to (113.0, 47.0)
- moved C3 82.0 mm to (119.4, 43.2)
- moved R3 81.7 mm to (110.5, 47.0)
- moved D2 81.5 mm to (115.6, 47.0)
- moved C4 79.2 mm to (123.2, 43.2), turned to 0 degrees
- moved D5 76.3 mm to (86.4, 55.9)
- moved U1 75.1 mm to (121.9, 49.5), turned to 270 degrees
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