File: ValveWizard The Engineers Thumb [5 knob]/ValveWizard The Engineers Thumb [5 knob].sch (KiCad schematic (older format))
At the start: 38 parts, among them Q1 ON_Semi_2N3906TAR, SW1 SW_BRIGHT, U1 TL072, U2 TL072, U3 LM13700

Commit message: Projects upd
Parts:
- Q1: symbol SA_Transistor_BJT:ON_Semi_2N3906TAR -> ValveWizard-The-Engineers-Thumb-[5-knob]-rescue:ON_Semi_2N3906TAR-SA_Transistor_BJT
- RV1, RV2, RV3, RV4, RV5: footprint SA_Potentiometers_THT:Alpha_Taiwan_9mm_Vertical -> SA_Potentiometers_THT:Alpha_Taiwan_RV16AF-10_THT
- U1, U2: symbol SA_Amplifiers_Operational:TL072 -> ValveWizard-The-Engineers-Thumb-[5-knob]-rescue:TL072-SA_Amplifiers_Operational
Connections:
- no-connect marks 1 -> 2
Changed lines of the file:
@@
 EESchema Schematic File Version 4
+LIBS:ValveWizard The Engineers Thumb [5 knob]-cache
 EELAYER 26 0
 EELAYER END
@@
 $EndComp
 $Comp
-L SA_Amplifiers_Operational:TL072 U1
+L ValveWizard-The-Engineers-Thumb-[5-knob]-rescue:TL072-SA_Amplifiers_Operational U1
 U 1 1 5C77CA56
 P 4950 3800
@@
 F 0 "RV2" V 5575 3600 50  0000 C CNN
 F 1 "1M" V 5650 3600 50  0000 C CNN
-F 2 "SA_Potentiometers_THT:Alpha_Taiwan_9mm_Vertical" H 5750 3600 50  0001 C CNN
+F 2 "SA_Potentiometers_THT:Alpha_Taiwan_RV16AF-10_THT" H 5750 3600 50  0001 C CNN
 F 3 "~" H 5750 3600 50  0001 C CNN
 	1    5750 3600
@@
 F 0 "RV5" V 8725 4050 50  0000 C CNN
 F 1 "10k" V 8800 4050 50  0000 C CNN
-F 2 "SA_Potentiometers_THT:Alpha_Taiwan_9mm_Vertical" H 8900 4050 50  0001 C CNN
+F 2 "SA_Potentiometers_THT:Alpha_Taiwan_RV16AF-10_THT" H 8900 4050 50  0001 C CNN
 F 3 "~" H 8900 4050 50  0001 C CNN
 	1    8900 4050
@@
 	8900 4400 8900 4200
 $Comp
-L SA_Amplifiers_Operational:TL072 U2
+L ValveWizard-The-Engineers-Thumb-[5-knob]-rescue:TL072-SA_Amplifiers_Operational U2
 U 2 1 5C7843C6
 P 4950 2100
@@
 F 0 "RV1" V 4325 2200 50  0000 C CNN
 F 1 "1M" V 4400 2200 50  0000 C CNN
-F 2 "SA_Potentiometers_THT:Alpha_Taiwan_9mm_Vertical" H 4500 2200 50  0001 C CNN
+F 2 "SA_Potentiometers_THT:Alpha_Taiwan_RV16AF-10_THT" H 4500 2200 50  0001 C CNN
 F 3 "~" H 4500 2200 50  0001 C CNN
 	1    4500 2200
@@
 F 0 "RV4" V 5675 2100 50  0000 C CNN
 F 1 "1M" V 5750 2100 50  0000 C CNN
-F 2 "SA_Potentiometers_THT:Alpha_Taiwan_9mm_Vertical" H 5850 2100 50  0001 C CNN
+F 2 "SA_Potentiometers_THT:Alpha_Taiwan_RV16AF-10_THT" H 5850 2100 50  0001 C CNN
 F 3 "~" H 5850 2100 50  0001 C CNN
 	1    5850 2100
@@
 F 0 "RV3" V 5675 1600 50  0000 C CNN
 F 1 "1M" V 5750 1600 50  0000 C CNN
-F 2 "SA_Potentiometers_THT:Alpha_Taiwan_9mm_Vertical" H 5850 1600 50  0001 C CNN
+F 2 "SA_Potentiometers_THT:Alpha_Taiwan_RV16AF-10_THT" H 5850 1600 50  0001 C CNN
 F 3 "~" H 5850 1600 50  0001 C CNN
 	1    5850 1600
@@
 $EndComp
 $Comp
-L SA_Amplifiers_Operational:TL072 U2
+L ValveWizard-The-Engineers-Thumb-[5-knob]-rescue:TL072-SA_Amplifiers_Operational U2
 U 1 1 5C7921EF
 P 6800 2000
@@
 $EndComp
 $Comp
-L SA_Transistor_BJT:ON_Semi_2N3906TAR Q1
+L ValveWizard-The-Engineers-Thumb-[5-knob]-rescue:ON_Semi_2N3906TAR-SA_Transistor_BJT Q1
 U 1 1 5C793C38
 P 7400 2000
@@
 Connection ~ 1600 6750
 $Comp
-L SA_Amplifiers_Operational:TL072 U1
+L ValveWizard-The-Engineers-Thumb-[5-knob]-rescue:TL072-SA_Amplifiers_Operational U1
 U 2 1 5C7BC1A7
 P 2250 6650
@@
 Text Notes 6200 4300 0    39   ~ 8
 Add no connects to unused OTA half
+NoConn ~ 7900 3000
 $EndSCHEMATC

Commit message: updated jfet matching scheme, eng. thumb. symbol rescue
Parts:
- Q1: symbol ValveWizard-The-Engineers-Thumb-[5-knob]-rescue:ON_Semi_2N3906TAR-SA_Transistor_BJT -> ValveWizard-The-Engineers-Thumb-[5-knob]-rescue:ON_Semi_2N3906TAR-SA_Transistor_BJT-ValveWizard-The-Engineers-Thumb-[5-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
- U1, U2: symbol ValveWizard-The-Engineers-Thumb-[5-knob]-rescue:TL072-SA_Amplifiers_Operational -> ValveWizard-The-Engineers-Thumb-[5-knob]-rescue:TL072-SA_Amplifiers_Operational-ValveWizard-The-Engineers-Thumb-[5-knob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
Changed lines of the file:
@@
 $EndComp
 $Comp
-L ValveWizard-The-Engineers-Thumb-[5-knob]-rescue:TL072-SA_Amplifiers_Operational U1
+L ValveWizard-The-Engineers-Thumb-[5-knob]-rescue:TL072-SA_Amplifiers_Operational-ValveWizard-The-Engineers-Thumb-[5-knob]-rescue U1
 U 1 1 5C77CA56
 P 4950 3800
@@
 	8900 4400 8900 4200
 $Comp
-L ValveWizard-The-Engineers-Thumb-[5-knob]-rescue:TL072-SA_Amplifiers_Operational U2
+L ValveWizard-The-Engineers-Thumb-[5-knob]-rescue:TL072-SA_Amplifiers_Operational-ValveWizard-The-Engineers-Thumb-[5-knob]-rescue U2
 U 2 1 5C7843C6
 P 4950 2100
@@
 $EndComp
 $Comp
-L ValveWizard-The-Engineers-Thumb-[5-knob]-rescue:TL072-SA_Amplifiers_Operational U2
+L ValveWizard-The-Engineers-Thumb-[5-knob]-rescue:TL072-SA_Amplifiers_Operational-ValveWizard-The-Engineers-Thumb-[5-knob]-rescue U2
 U 1 1 5C7921EF
 P 6800 2000
@@
 $EndComp
 $Comp
-L ValveWizard-The-Engineers-Thumb-[5-knob]-rescue:ON_Semi_2N3906TAR-SA_Transistor_BJT Q1
+L ValveWizard-The-Engineers-Thumb-[5-knob]-rescue:ON_Semi_2N3906TAR-SA_Transistor_BJT-ValveWizard-The-Engineers-Thumb-[5-knob]-rescue Q1
 U 1 1 5C793C38
 P 7400 2000
@@
 Connection ~ 1600 6750
 $Comp
-L ValveWizard-The-Engineers-Thumb-[5-knob]-rescue:TL072-SA_Amplifiers_Operational U1
+L ValveWizard-The-Engineers-Thumb-[5-knob]-rescue:TL072-SA_Amplifiers_Operational-ValveWizard-The-Engineers-Thumb-[5-knob]-rescue U1
 U 2 1 5C7BC1A7
 P 2250 6650
