File: Switching_Scheme_Prototype_40106_SMD/Switching_Scheme_Prototype_40106_SMD.sch (KiCad schematic (older format))
At the start: 22 parts, among them J2 Neutrik_NRJ6HM-1, J3 SEND, J4 Neutrik_NRJ6HM-1, J5 RETURN, K1 EA2-5SNJ, Q3 MBT3946DW1T1G, SW1 Momentary_NO, U1 Texas_Instruments_CD40106BPWR

Commit message: Update Switching_Scheme_Prototype_40106_SMD.sch
Parts:
- C1: value 0.1 -> 4n7
- C2: value 0.22 -> 47n
Other:
- note added: "CRITICAL"
- note added: "Test 390R resistor with 10k trimpot for LED"
- note added: "Test separate inverter for LED current sink"
- moved on the sheet: C4, D2, R3, R7, U1F
Changed lines of the file:
@@
 P 1125 2900
 F 0 "C1" H 1150 3000 39  0000 L CNB
-F 1 "0.1" H 1150 3050 20  0000 L CNB
+F 1 "4n7" H 1150 3050 20  0000 L CNB
 F 2 "SA_Capacitors_SMD:C_0603_1608M" H 1050 2900 20  0001 C CNN
 F 3 "~" H 1125 2900 50  0001 C CNN
@@
 P 1825 2900
 F 0 "C2" H 1850 3000 39  0000 L CNB
-F 1 "0.22" H 1850 3050 20  0000 L CNB
+F 1 "47n" H 1850 3050 20  0000 L CNB
 F 2 "SA_Capacitors_SMD:C_0603_1608M" H 1750 2900 20  0001 C CNN
 F 3 "~" H 1825 2900 50  0001 C CNN
@@
 L Device:LED_ALT D2
 U 1 1 5C4E6D21
-P 3225 2100
-F 0 "D2" H 3225 2200 39  0000 C CNB
-F 1 "LED" H 3225 2000 20  0000 C CNB
-F 2 "SA_Connectors_Pin_Headers_THT:PinHeader_1x02_P2.54mm_Vertical_Top" H 3225 2100 50  0001 C CNN
-F 3 "~" H 3225 2100 50  0001 C CNN
-	1    3225 2100
+P 3225 1400
+F 0 "D2" H 3225 1500 39  0000 C CNB
+F 1 "LED" H 3225 1300 20  0000 C CNB
+F 2 "SA_Connectors_Pin_Headers_THT:PinHeader_1x02_P2.54mm_Vertical_Top" H 3225 1400 50  0001 C CNN
+F 3 "~" H 3225 1400 50  0001 C CNN
+	1    3225 1400
 	0    -1   -1   0
 $EndComp
@@
 L SA_Device:R R3
 U 1 1 5CB98594
-P 3225 1450
-F 0 "R3" V 3305 1450 39  0000 C CNB
-F 1 "CLR-A" V 3225 1450 20  0000 C CNB
-F 2 "SA_Capacitors_SMD:C_0603_1608M" V 3155 1450 50  0001 C CNN
-F 3 "" H 3225 1450 50  0001 C CNN
-	1    3225 1450
+P 3225 750
+F 0 "R3" V 3305 750 39  0000 C CNB
+F 1 "CLR-A" V 3225 750 20  0000 C CNB
+F 2 "SA_Capacitors_SMD:C_0603_1608M" V 3155 750 50  0001 C CNN
+F 3 "" H 3225 750 50  0001 C CNN
+	1    3225 750
 	1    0    0    -1
 $EndComp
@@
 L SA_CMOS_Logic:Texas_Instruments_CD40106BPWR U1
 U 6 1 5CBE4732
-P 2100 4025
-F 0 "U1" H 2150 4175 39  0000 L CNB
-F 1 "Texas_Instruments_CD40106BPWR" H 2150 4225 20  0000 L CNB
-F 2 "SA_CMOS_Logic_SMD:Texas_Instruments_CD40106BPWR_TSSOP-14" H 2100 4025 20  0001 C CNN
-F 3 "https://www.onsemi.com/pub/Collateral/NL37WZ14-D.PDF" H 2150 4025 50  0001 C CNN
-	6    2100 4025
+P 2875 1750
+F 0 "U1" H 2925 1900 39  0000 L CNB
+F 1 "Texas_Instruments_CD40106BPWR" H 2925 1950 20  0000 L CNB
+F 2 "SA_CMOS_Logic_SMD:Texas_Instruments_CD40106BPWR_TSSOP-14" H 2875 1750 20  0001 C CNN
+F 3 "https://www.onsemi.com/pub/Collateral/NL37WZ14-D.PDF" H 2925 1750 50  0001 C CNN
+	6    2875 1750
 	1    0    0    -1
 $EndComp
@@
 L SA_Power:VCC #PWR010
 U 1 1 5CBF4543
-P 3225 1300
-F 0 "#PWR010" H 3225 1150 50  0001 C CNN
-F 1 "VCC" H 3225 1450 39  0000 C CNB
-F 2 "" H 3225 1300 50  0001 C CNN
-F 3 "" H 3225 1300 50  0001 C CNN
-	1    3225 1300
+P 3225 600
+F 0 "#PWR010" H 3225 450 50  0001 C CNN
+F 1 "VCC" H 3225 750 39  0000 C CNB
+F 2 "" H 3225 600 50  0001 C CNN
+F 3 "" H 3225 600 50  0001 C CNN
+	1    3225 600
 	1    0    0    -1
 $EndComp
@@
 L SA_Device:R R7
 U 1 1 5CBF482C
-P 3225 1800
-F 0 "R7" V 3305 1800 39  0000 C CNB
-F 1 "CLR-B" V 3225 1800 20  0000 C CNB
-F 2 "SA_Capacitors_SMD:C_0603_1608M" V 3155 1800 50  0001 C CNN
-F 3 "" H 3225 1800 50  0001 C CNN
-	1    3225 1800
-	1    0    0    -1
-$EndComp
-Wire Wire Line
-	3225 1600 3225 1625
+P 3225 1100
+F 0 "R7" V 3305 1100 39  0000 C CNB
+F 1 "CLR-B" V 3225 1100 20  0000 C CNB
+F 2 "SA_Capacitors_SMD:C_0603_1608M" V 3155 1100 50  0001 C CNN
+F 3 "" H 3225 1100 50  0001 C CNN
+	1    3225 1100
+	1    0    0    -1
+$EndComp
+Wire Wire Line
+	3225 900  3225 925
 $Comp
 L SA_Capacitors:Nichicon_UWT_100uF_25V C4
 U 1 1 5CBF6530
-P 2850 1800
-F 0 "C4" V 3000 1750 39  0000 L CNB
-F 1 "10/25" V 3050 1750 20  0000 L CNB
-F 2 "Capacitor_Tantalum_SMD:CP_EIA-6032-28_Kemet-C" H 2775 1800 20  0001 C CNN
-F 3 "~" H 2850 1800 50  0001 C CNN
-	1    2850 1800
-	1    0    0    -1
-$EndComp
-Wire Wire Line
-	2850 1650 2850 1625
-Wire Wire Line
-	2850 1625 3225 1625
-Connection ~ 3225 1625
-Wire Wire Line
-	3225 1625 3225 1650
+P 2850 1125
+F 0 "C4" V 3000 1075 39  0000 L CNB
+F 1 "10/25" V 3050 1075 20  0000 L CNB
+F 2 "Capacitor_Tantalum_SMD:CP_EIA-6032-28_Kemet-C" H 2775 1125 20  0001 C CNN
+F 3 "~" H 2850 1125 50  0001 C CNN
+	1    2850 1125
+	1    0    0    -1
+$EndComp
+Wire Wire Line
+	2850 975  2850 950
+Wire Wire Line
+	2850 925  3225 925
+Connection ~ 3225 925
+Wire Wire Line
+	3225 925  3225 950
 $Comp
 L SA_Power:GND #PWR011
 U 1 1 5CBF838C
-P 2850 1950
-F 0 "#PWR011" H 2850 1700 50  0001 C CNN
-F 1 "GND" H 2850 1800 39  0000 C CNB
-F 2 "" H 2850 1950 50  0001 C CNN
-F 3 "" H 2850 1950 50  0001 C CNN
-	1    2850 1950
-	1    0    0    -1
-$EndComp
+P 2850 1275
+F 0 "#PWR011" H 2850 1025 50  0001 C CNN
+F 1 "GND" H 2850 1125 39  0000 C CNB
+F 2 "" H 2850 1275 50  0001 C CNN
+F 3 "" H 2850 1275 50  0001 C CNN
+	1    2850 1275
+	1    0    0    -1
+$EndComp
+Text Notes 1350 3700 0    50   Italic 10
+CRITICAL
+Text Notes 3400 1250 0    50   Italic 10
+Test 390R resistor with 10k trimpot for LED
+Text Notes 3425 1525 0    50   Italic 10
+Test separate inverter for LED current sink
 $EndSCHEMATC
