File: Musitronics Mu-Tron II Phaser/Factory Schematic/Musitronics MuTron Phasor II Factory Schematic/Musitronics MuTron Phasor II Factory Schematic.sch (KiCad schematic (older format))
At the start: 68 parts, among them U1 RC4558, U2 RC4558, U3 RC4558, U4 RC4558, U5 RC4558

Commit message: Revert "edit computer 2"
This reverts commit 52804b7d86e33d0668af1082d22f36fcd7cbbfe3.
Parts:
- removed C16: 470n, symbol Musitronics-MuTron-Phasor-II-Factory-Schematic-rescue:C-SA_Device
- removed C23: 6n8, symbol Musitronics-MuTron-Phasor-II-Factory-Schematic-rescue:C-SA_Device
- removed R33: 56k, symbol Musitronics-MuTron-Phasor-II-Factory-Schematic-rescue:R-SA_Device
- removed R34: 82R, symbol Musitronics-MuTron-Phasor-II-Factory-Schematic-rescue:R-SA_Device
- removed R35, R57: 27k, symbol Musitronics-MuTron-Phasor-II-Factory-Schematic-rescue:R-SA_Device
- removed R54: 10k (DEPTH), symbol Musitronics-MuTron-Phasor-II-Factory-Schematic-rescue:R_POT-SA_Device
- removed R55: 25k (RATE), symbol Musitronics-MuTron-Phasor-II-Factory-Schematic-rescue:R_POT-SA_Device
- removed R56: 100k, symbol Musitronics-MuTron-Phasor-II-Factory-Schematic-rescue:R-SA_Device
- removed U? (x2): RC4558-SA_Amplifiers_Operational, symbol Musitronics-MuTron-Phasor-II-Factory-Schematic-rescue:RC4558-SA_Amplifiers_Oper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
- 4k7, R1, R10, R11, R12, R13, R14, R15, R16, R17, R18, R19, R20, R21, R22, R23, R24, R25, R26, R27, R28, R29, R3, R30, R31, R5, R6, R7, R8, R9: symbol Musitronics-MuTron-Phasor-II-Factory-Schematic-rescue:R-SA_Device -> SA_Device:R
- C1, C10, C11, C12, C14, C15, C2, C3, C4, C5, C6, C7, C8, C9: symbol Musitronics-MuTron-Phasor-II-Factory-Schematic-rescue:C-SA_Device -> SA_Device:C
- C13: symbol Musitronics-MuTron-Phasor-II-Factory-Schematic-rescue:CP1-SA_Device -> SA_Device:CP1
- PM1A, PM1B, PM1C, PM1D, PM1E, PM1F: symbol Musitronics-MuTron-Phasor-II-Factory-Schematic-rescue:R_PHOTO-SA_Device -> SA_Device:R_PHOTO
- R53: symbol Musitronics-MuTron-Phasor-II-Factory-Schematic-rescue:R_POT-SA_Device -> SA_Device:R_POT
- U1, U2, U3, U4, U5: symbol Musitronics-MuTron-Phasor-II-Factory-Schematic-rescue:RC4558-SA_Amplifiers_Operational -> SA_Amplifiers_Operational:RC4558
Connections:
- net at C6.1, U2.3 (+): no longer PM1A.1, R10.2
- net at C7.1, U2.5 (+): no longer PM1B.1, R13.2
- net at C8.1, U3.3 (+): no longer PM1C.1, R16.2
- net at C9.1, U3.5 (+): no longer PM1D.1, R19.2
- net at C10.1, U4.3 (+): no longer PM1E.1, R22.2
- net at C11.1, U4.5 (+): no longer PM1F.1, R25.2
- now unconnected: PM1A.2, PM1B.2, PM1C.2, PM1D.2, PM1E.2, PM1F.2, R10.1, R13.1, R16.1, R19.1, R22.1, R25.1
Other:
- moved on the sheet: 4k7, C1, C10, C11, C12, C13, C14, C15, C2, C3, C4, C5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

Commit message: edit computer 2
Parts:
- added C16: 470n, symbol Musitronics-MuTron-Phasor-II-Factory-Schematic-rescue:C-SA_Device
- added C23: 6n8, symbol Musitronics-MuTron-Phasor-II-Factory-Schematic-rescue:C-SA_Device
- added R33: 56k, symbol Musitronics-MuTron-Phasor-II-Factory-Schematic-rescue:R-SA_Device
- added R34: 82R, symbol Musitronics-MuTron-Phasor-II-Factory-Schematic-rescue:R-SA_Device
- added R35, R57: 27k, symbol Musitronics-MuTron-Phasor-II-Factory-Schematic-rescue:R-SA_Device
- added R54: 10k (DEPTH), symbol Musitronics-MuTron-Phasor-II-Factory-Schematic-rescue:R_POT-SA_Device
- added R55: 25k (RATE), symbol Musitronics-MuTron-Phasor-II-Factory-Schematic-rescue:R_POT-SA_Device
- added R56: 100k, symbol Musitronics-MuTron-Phasor-II-Factory-Schematic-rescue:R-SA_Device
- added U? (x2): RC4558-SA_Amplifiers_Operational, symbol Musitronics-MuTron-Phasor-II-Factory-Schematic-rescue:RC4558-SA_Amplifiers_Oper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
- 4k7, R1, R10, R11, R12, R13, R14, R15, R16, R17, R18, R19, R20, R21, R22, R23, R24, R25, R26, R27, R28, R29, R3, R30, R31, R5, R6, R7, R8, R9: symbol SA_Device:R -> Musitronics-MuTron-Phasor-II-Factory-Schematic-rescue:R-SA_Device
- C1, C10, C11, C12, C14, C15, C2, C3, C4, C5, C6, C7, C8, C9: symbol SA_Device:C -> Musitronics-MuTron-Phasor-II-Factory-Schematic-rescue:C-SA_Device
- C13: symbol SA_Device:CP1 -> Musitronics-MuTron-Phasor-II-Factory-Schematic-rescue:CP1-SA_Device
- PM1A, PM1B, PM1C, PM1D, PM1E, PM1F: symbol SA_Device:R_PHOTO -> Musitronics-MuTron-Phasor-II-Factory-Schematic-rescue:R_PHOTO-SA_Device
- R53: symbol SA_Device:R_POT -> Musitronics-MuTron-Phasor-II-Factory-Schematic-rescue:R_POT-SA_Device
- U1, U2, U3, U4, U5: symbol SA_Amplifiers_Operational:RC4558 -> Musitronics-MuTron-Phasor-II-Factory-Schematic-rescue:RC4558-SA_Amplifiers_Operational
Connections:
- net at C6.1, U2.3 (+): now also PM1A.1, R10.2
- net at C7.1, U2.5 (+): now also PM1B.1, R13.2
- net at R10.1: now also PM1A.2, PM1B.2, PM1C.2, PM1D.2, PM1E.2, PM1F.2, R13.1, R16.1, R19.1, R22.1, R25.1
- net at C8.1, U3.3 (+): now also PM1C.1, R16.2
- net at C9.1, U3.5 (+): now also PM1D.1, R19.2
- net at C10.1, U4.3 (+): now also PM1E.1, R22.2
- net at C11.1, U4.5 (+): now also PM1F.1, R25.2
- new net: C23.2, R56.1, U?.2 (-)
- new net: C23.1, R33.1, R55.3, U?.1
- new net: R33.2, U?.3 (+)
- new net: R34.2, R55.1
- new net: R35.2, R55.2
- new net: C16.2, R35.1, U?.6 (-)
- new net: R57.2, U?.5 (+)
- new net: C16.1, R54.3, U?.7
Other:
- moved on the sheet: 4k7, C1, C10, C11, C12, C13, C14, C15, C2, C3, C4, C5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
